File: Circuito/PlacaAquisicao/PlacaAquisicao.sch (EAGLE design)
At the start: 98 parts, among them IC2 LM7805, IC3 MEGA8-AI, IC4 ACS712-LC, IC5 MEGA8-AI, IC6 ACS712-LC, IC7 MCP602P, IC8 MCP602P, P1 SPI, P2 SPI, Q1 16MHz, X1 MC4-G, X2 MC4-G, X3 MSTBA2, X4 MSTBA2, X6 MC4-G, X7 MC4-G

Commit message: Atualizando...
Parts:
- added C34: 4,7uF, rcl:CPOL-EUE2.5-6
- added C35: 100uF 50V, rcl:CPOL-USE2.5-7
- added C38: 470uF 16V, rcl:CPOL-USE2.5-7
- added D3: SS56, ,RK_SteveMarple:DIODE-SCHOTTKY_
- added IC1: REG1117, burr-brown:REG1117
- added IC10: (no value), linear:LM2596S
- added L2: 100uH, inductors:DR125
- added R3, R42: 560, rcl:R-EU_0207/7
- added R41: 120, rcl:R-EU_0207/7
- added R43, R45: 1K, rcl:R-EU_0207/7
- added R44: 10K, rcl:R-EU_0207/7
- added R46: 11.3K, rcl:R-EU_0207/7
- added X5, X8: MC4-G, con-phoenix-381_l:MC4-G
- IC2: value LM7805 -> LTC485S; device v-reg:78XXL -> linear-technology:LTC485S
- R10, R12, R14, R16, R18, R20, R22, R24, R26, R4, R6, R8: value 8,3K -> 9,1K
Connections:
- removed net N$20: R26.2, X7.2.SK
- new net +15V: C38.+, L2.2, R46.2, X8.4.SK
- new net N$35: R43.2, R44.2, X5.3.SK
- new net N$36: IC10.FB, R45.2, R46.1
- new net N$37: D3.C, IC10.OUT, L2.1
- new net N$5: IC3.PB2(SS/OC1B), IC5.PB2(SS/OC1B)
- new net RS485A: IC2.A, R3.1, R41.2, X7.2.SK
- new net RS485B: IC2.B, R41.1, R42.2, X7.3.SK
- new net RXD: IC2.RO, IC3.PD0(RXD)
- new net TEMP_IN: C34.+, IC5.PC4(ADC4/SDA), R44.1
- new net TXD: IC2.DI, IC3.PD1(TXD)
- new net TXE: IC2.!RE, IC2.DE, IC3.PD4(XCK/T0)
- new net VC10: R22.2, X6.3.SK
- net +5V: now also IC1.VOUT, IC2.VCC, R3.2, X5.1.SK, X5.2.SK; no longer IC2.OUT
- net +8V: now also IC1.VIN, X8.3.SK; no longer IC2.IN
- net ADC0A: now also C10.+, R12.1, R13.2; no longer C13.+, R18.1, R19.2
- net ADC1A: now also C11.+, R14.1, R15.2; no longer C12.+, R16.1, R17.2
- net ADC2A: now also C12.+, R16.1, R17.2; no longer C11.+, R14.1, R15.2
- net ADC3A: now also C13.+, R18.1, R19.2; no longer C10.+, R12.1, R13.2
- net ADC4A: now also C14.+, R20.1, R21.2; no longer C9.+, R10.1, R11.2
- net ADC5A: now also C15.+, R22.1, R23.2; no longer C8.+, R8.1, R9.2
- net ADC6A: now also C8.+, R8.1, R9.2; no longer C15.+, R22.1, R23.2
- net ADC7A: now also C9.+, R10.1, R11.2; no longer C14.+, R20.1, R21.2
- net GND: now also C34.-, C35.-, C38.-, D3.A, IC1.GND, IC10.EN, IC10.GND, IC10.GND@1, R42.1, R43.1, R45.1, X5.4.SK, X7.4.SK, X8.2.SK
- net N$1: now also C35.+, IC10.IN
- net N$10: now also R26.2; no longer X6.3.SK
- net N$11: now also X4-2.1; no longer X4-1.1
- net N$12: now also X4-1.1; no longer X4-2.1
- net N$18: now also X3-1.1; no longer X3-2.1
- net N$21: now also X7.1.SK; no longer X7.3.SK
- net N$33: now also JP1.4; no longer JP1.6
- net N$34: now also JP1.6; no longer JP1.4
- net N$9: now also X3-2.1; no longer X3-1.1
- net VIN: now also X8.1.SK; no longer R22.2, X7.1.SK
Other:
- note added: "LM35"
- moved on the sheet: C18, C19, C20, C21, C22, C23, C26, C27, C28, C29, C3, C30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

Commit message: versão 2022
Connections:
- new net N$20: IC3.PD3(INT1), X5.1.SK
- net +5V: no longer X5.1.SK
Other:
- note added: "Controle"
- note added: "Corrente + (in)"
- note added: "Corrente - (out)"
- note added: "Display"
- note added: "GND"
- note added: "Motor"
- note added: "Módulo"
- note added: "Placa Telemetria"
- note added: "RS485-A"
- note added: "RS485-B"
- note added: "Reserva"
- note added: "Rádio"
- note added: "Sensor"
- note added: "Temperatura"
- note added: "V2.0"
- note added: "Vc1"
- note added: "Vc10"
- note added: "Vc11"
- note added: "Vc12"
- note added: "Vc2"
- note added: "Vc3"
- note added: "Vc4"
- note added: "Vc5"
- note added: "Vc6"
- note added: "Vc7"
- note added: "Vc8"
- note added: "Vc9"
- note added: "Velocidade"
- note added: "Vin(42V)"
- note added: "Volante"
- note added: "Vout 15V"
- note added: "Vout 5V"
- note added: "Vout 8V"
- note added: "de"
- note added: "do"
- moved on the sheet: X5.1
